File: Hardware/0. Project/DrizzlingBytes.sch (EAGLE design)
At the start: 35 parts, among them CN1 USB Type C Receptacle, Q1 NPN-BC817, Q2 NPN-BC817, Q3 NPN-BC817, U1 CP2102N, U2 1117-3.3V, U3 MSP430FR4133

Commit message: Schematic v1.1 release
Connections:
- new net N$15: Q2.B, R6.2
- net USB_RTS: no longer Q2.B, R6.2
Other:
- note added: "V1.1 - BUG fix: changed R6 position to protects Q2 BJT's base."
- note added: "v1.0 - Initial Release"
